Commit message: Update tatacoa.transmission.xacro

File: tatacoa_ws/src/tatacoa_description/URDF/tatacoa.transmission.xacro (robot description, xacro)
@@ -21,5 +21,5 @@
           rpy="0 0 ${0.5*pi*(reflect+1)}" />
         <geometry>
-          <mesh filename="package://bogbot_description/meshes/wheel_bogbot.dae" />
+          <mesh filename="package://tatacoa_description/meshes/wheel_bogbot.dae" />
         </geometry>
       </visual>
@@ -58,5 +58,5 @@
         <origin xyz="-0.4365 ${reflect*0.23} -0.025" rpy="0 0 ${-reflect*pi/4}" />
         <geometry>
-          <mesh filename="package://bogbot_description/meshes/caster_wheel.dae" />
+          <mesh filename="package://tatacoa_description/meshes/caster_wheel.dae" />
         </geometry>
       </visual>
