Commit message: Update tatacoa.urdf.xacro

File: tatacoa_ws/src/tatacoa_description/URDF/tatacoa.urdf.xacro (robot description, xacro)
@@ -1,75 +1,68 @@
 <?xml version="1.0"?>
-<robot xmlns:xacro="http://ros.org/wiki/xacro" name="robot_essentials" >
-  <!--######################################################################-->
-  <xacro:macro name="wheel" params="prefix reflect mass radius length">
-    <!-- LINK -->
-    <link name="${prefix}_wheel">
-      <inertial>
-        <origin xyz="0 0 0" rpy="0 0 0" />
-        <mass value="${mass}" />
-        <inertia
-          ixx="${0.0833333 * mass * (3 * radius * radius + length * length)}"
-          ixy="0.0"
-          ixz="0.0"
-          iyy="${0.0833333 * mass * (3 * radius * radius + length * length)}"
-          iyz="0.0"
-          izz="${0.5 * mass * radius * radius}" />
-      </inertial>
-      <visual>
-        <origin
-          xyz="0 0 0"
-          rpy="0 0 ${0.5*pi*(reflect+1)}" />
-        <geometry>
-          <mesh filename="package://tatacoa_description/meshes/wheel_bogbot.dae" />
-        </geometry>
-      </visual>
-      <collision>
-        <origin
-          xyz="0 0 0"
-          rpy="${pi/2} 0 0" />
-        <geometry>
-          <cylinder length="${length}" radius="${radius}"/>
-        </geometry>
-      </collision>
-    </link>
-    <!--JOINT-->
-    <joint name="${prefix}_wheel_joint" type="continuous">
-      <axis xyz="0 1 0"/>
-      <parent link ="base_link"/>
-      <child link ="${prefix}_wheel"/>
-      <origin rpy ="0 0 0" xyz= "-0.01 ${reflect*0.29} -0.05"/>
-    </joint>
-    <!--TRANSMISSION -->
-    <transmission name="${prefix}_wheel_trans" type="SimpleTransmission">
-      <type>transmission_interface/SimpleTransmission</type>
-      <actuator name="${prefix}_wheel_motor">
-        <hardwareInterface>hardware_interface/VelocityJointInterface</hardwareInterface>
-        <mechanicalReduction>1</mechanicalReduction>
-      </actuator>
-      <joint name="${prefix}_wheel_joint">
-        <hardwareInterface>hardware_interface/VelocityJointInterface</hardwareInterface>
-      </joint>
-    </transmission>
-  </xacro:macro>
-  <!-- Macro for defining caster wheels -->
-  <xacro:macro name="caster_wheel" params="prefix reflect radius">
-    <link name="${prefix}_caster_wheel">
-      <visual>
-        <origin xyz="-0.4365 ${reflect*0.23} -0.025" rpy="0 0 ${-reflect*pi/4}" />
-        <geometry>
-          <mesh filename="package://tatacoa_description/meshes/caster_wheel.dae" />
-        </geometry>
-      </visual>
-      <collision>
-        <origin xyz="-0.4365 ${reflect*0.25} -0.06" rpy="0 0 0" />
-        <geometry>
-          <sphere radius="${radius}"/>
-        </geometry>
-      </collision>
-    </link>
-    <joint name="${prefix}_caster_wheel_joint" type="fixed">
-      <parent link="base_link"/>
-      <child link="${prefix}_caster_wheel"/>
-    </joint>
-  </xacro:macro>
+<robot xmlns:xacro="http://wiki.ros.org/xacro" name="tatacoa">
+  <xacro:property name="mass_base" value="10" />
+  <xacro:property name="mass_wheel" value="10" />
+  <xacro:property name="wheel_r" value="0.05" />
+  <xacro:property name="wheel_r_2_top" value="0.05" />
+  <xacro:property name="name_lidar" value="rplidar" />
+  <xacro:property name="origin_lidar" value="0.1065 0.0 0.07"/>
+  <xacro:include filename="$(find bogbot_description)/urdf/tatacoa.transmission.xacro" />
+  <xacro:include filename="$(find bogbot_description)/urdf/tatacoa.gazebo.xacro" />
+    <!-- Robot base_link -->
+  <link name="base_link">
+    <visual>
+      <origin rpy="0 0 0" xyz="0 0 0"/>
+      <geometry>
+        <mesh filename="package://tatacoa_description/meshes/base_robot.dae"/>
+      </geometry>
+    </visual>
+    <visual>
+      <origin rpy="0 0 0" xyz="0.17 0 0"/>
+      <geometry>
+        <mesh filename="package://tatacoa_description/meshes/cover_msg.dae"/>
+      </geometry>
+    </visual>
+    <collision>
+      <origin rpy="0 0 0" xyz="-0.1235 0 0"/>
+      <geometry>
+        <box size="0.7 0.55 0.1"/>
+      </geometry>
+    </collision>
+    <inertial>
+      <mass value="${mass_base}"/>
+      <origin xyz="-0.1235 0 -0.05" />
+      <inertia ixx="${0.0833333 * mass_base * (0.5*0.5 + 0.1*0.1)}" ixy="0.0" ixz="0.0"
+        iyy="${0.0833333 * mass_base * (0.6*0.6 + 0.1*0.1)}" iyz="0.0"
+        izz="${0.0833333 * mass_base * (0.6*0.6 + 0.5*0.5)}" />
+    </inertial>
+  </link>
+  <!-- Fixed offset from the floor to the center of the wheels -->
+  <link name="base_footprint"/>
+  <joint name="base_footprint_joint" type="fixed">
+    <parent link="base_footprint"/>
+    <child link="base_link"/>
+    <origin xyz="0 0 ${wheel_r_2_top+wheel_r}" rpy="0 0 0"/>
+  </joint>
+  <xacro:wheel prefix="left" reflect="1" mass="${mass_wheel}" radius="${wheel_r}" length="0.05"/>
+  <xacro:wheel prefix="right" reflect="-1" mass="${mass_wheel}" radius="${wheel_r}" length="0.05"/>
+  <xacro:caster_wheel prefix="left" reflect="1"  radius="0.035"/>
+  <xacro:caster_wheel prefix="right" reflect="-1"  radius="0.035"/>
+  <!-- Lidar -->
+  <link name="${name_lidar}_link">
+    <visual>
+      <origin xyz="0 0 -0.025" rpy="${pi/2} 0 ${pi/2}"/>
+      <geometry>
+        <mesh filename="package://tatacoa_description/meshes/rplidar_A2.dae" scale="0.001 0.001 0.001"/>
+      </geometry>
+    </visual>
+  </link>
+  <joint name="${name_lidar}_joint" type="fixed">
+    <parent link="base_link"/>
+    <child link="${name_lidar}_link"/>
+    <origin xyz="${origin_lidar}" rpy="0 0 0"/>
+  </joint>
+  <!-- Camera -->
+  <xacro:realsense_T265 sensor_name="camera" parent_link="base_link" rate="30.0">
+    <origin rpy="0 0 0" xyz="0.18 0 0.0"/>
+  </xacro:realsense_T265>
 </robot>
